Commit message: full package

File: install/rmitbot_description/share/rmitbot_description/urdf/rmitbot.urdf.xacro (robot description, xacro)
@@ -1,11 +1,10 @@
 <?xml version="1.0"?>
-<robot name="rmitbot"
-    xmlns:xacro="http://ros.org/wiki/xacro">
-    <!-- Load Simulated or Real Hardware Interfaces -->
-    <xacro:arg name="is_sim" default="true"/>
+<!-- This is the main urdf document, calling other xacro, including -->
+<!-- rmitbot_platform:  main platform -->
+<!-- rmitbot_gazebo:    gazebo simulation parameters for the main platform -->
+<robot name="rmitbot" xmlns:xacro="http://ros.org/wiki/xacro">
+    <!-- Include Gazebo Parameters -->
     <xacro:include filename="$(find rmitbot_description)/urdf/rmitbot_platform.xacro" />
     <xacro:include filename="$(find rmitbot_description)/urdf/rmitbot_gazebo.xacro" />
     <xacro:include filename="$(find rmitbot_description)/urdf/rmitbot_ros2_control.xacro" />
-    <xacro:include filename="$(find rmitbot_description)/urdf/rmitbot_imu.xacro" />
-    <xacro:include filename="$(find rmitbot_description)/urdf/rmitbot_laser.xacro" />
 </robot>

File: install/rmitbot_description/share/rmitbot_description/urdf/rmitbot_gazebo.xacro (robot description, xacro)
@@ -1,6 +1,7 @@
 <?xml version="1.0"?>
+<!-- Gazebo file contains information regarding the lnks's physics (e.g., friction, stiffness, damping) -->
 <robot name="rmitbot" xmlns:xacro="http://ros.org/wiki/xacro">
   <!-- Wheels -->
-  <gazebo reference="wheel_left_link">
+  <gazebo reference="front_right_wheel">
     <mu1>1000000000000000.0</mu1>
     <mu2>1000000000000000.0</mu2>
@@ -11,5 +12,5 @@
     <fdir1>1 0 0</fdir1>
   </gazebo>
-  <gazebo reference="wheel_right_link">
+  <gazebo reference="front_left_wheel">
     <mu1>1000000000000000.0</mu1>
     <mu2>1000000000000000.0</mu2>
@@ -20,20 +21,21 @@
     <fdir1>1 0 0</fdir1>
   </gazebo>
-  <!-- Caster Wheels -->
-  <gazebo reference="caster_rear_link">
-    <mu1>0.1</mu1>
-    <mu2>0.1</mu2>
-    <kp>1000000.0</kp>
-    <kd>100.0</kd>
+  <gazebo reference="rear_right_wheel">
+    <mu1>1000000000000000.0</mu1>
+    <mu2>1000000000000000.0</mu2>
+    <kp>1000000000000.0</kp>
+    <kd>10.0</kd>
     <minDepth>0.001</minDepth>
-    <maxVel>1.0</maxVel>
+    <maxVel>0.1</maxVel>
+    <fdir1>1 0 0</fdir1>
   </gazebo>
-  <gazebo reference="caster_front_link">
-    <mu1>0.1</mu1>
-    <mu2>0.1</mu2>
-    <kp>1000000.0</kp>
-    <kd>100.0</kd>
+  <gazebo reference="rear_left_wheel">
+    <mu1>1000000000000000.0</mu1>
+    <mu2>1000000000000000.0</mu2>
+    <kp>1000000000000.0</kp>
+    <kd>10.0</kd>
     <minDepth>0.001</minDepth>
-    <maxVel>1.0</maxVel>
+    <maxVel>0.1</maxVel>
+    <fdir1>1 0 0</fdir1>
   </gazebo>
 </robot>

File: install/rmitbot_description/share/rmitbot_description/urdf/rmitbot_platform.xacro (robot description, xacro)
@@ -8,18 +8,27 @@
     <link name="base_link">
         <inertial>
-            <origin xyz="0 0 0.04" rpy="0.0 0.25 0.3" />
-            <mass value="8.2573504e-01"/>
-            <inertia ixx="2.2124416e-02" ixy="-1.2294101e-04" ixz="3.4938785e-04" iyy="2.1193702e-02" iyz="-5.0120904e-05" izz="2.0064271e-02" />
+            <origin xyz="0 0 0" rpy="0.0 0.0 0.0" />
+            <mass value="3.824"/>
+            <inertia
+                ixx="0.092" ixy="0.02" ixz="-5.178e-05"
+                iyy="0.061" iyz="0"
+                izz="0.145" />
         </inertial>
         <visual>
-            <origin xyz="0 0 0" rpy="0 0 0" />
+            <origin xyz="0 0 -0.002" rpy="0 0 0" />
             <geometry>
-                <mesh filename="package://rmitbot_description/meshes/base_link.STL" />
+                <mesh filename="package://rmitbot_description/meshes/base_link.stl" scale="0.001 0.001 0.001"/>
             </geometry>
         </visual>
         <collision>
-            <origin xyz="0 0 0" rpy="0 0 0" />
+            <origin xyz="0 0 0.068" rpy="0 0 0" />
             <geometry>
-                <mesh filename="package://rmitbot_description/meshes/base_link.STL" />
+                <box size="0.40 0.38 0.03"/>
+            </geometry>
+        </collision>
+        <collision>
+            <origin xyz="0 0 0.023" rpy="0 0 0" />
+            <geometry>
+                <box size="0.30 0.38 0.065"/>
             </geometry>
         </collision>
@@ -28,105 +37,117 @@
         <parent link="base_footprint"/>
         <child link="base_link" />
-        <origin xyz="0 0 0.033" rpy="0 0 0"/>
+        <origin xyz="0 0 0.052" rpy="0 0 0"/>
     </joint>
-    <link name="wheel_right_link">
+    <link name="front_left_wheel">
         <inertial>
-            <origin xyz="0 -0.014 0" rpy="0 0 0" />
-            <mass value="0.0530086090966721" />
-            <inertia ixx="1.88176298336665E-05" ixy="-4.8444933029987E-10" ixz="1.88163708851143E-08" iyy="3.11510738647764E-05" iyz="-6.93560663069607E-11" izz="1.8801969558182E-05" />
+            <origin xyz="0 0 0" rpy="0 0 0" />
+            <mass value="4.315763" />
+            <inertia
+                ixx="5.3947033e-03" ixy="6.821e-17" ixz="-1.137e-17"
+                iyy="4.4596211e-03" iyz="0.0"
+                izz="4.4596218e-03" />
         </inertial>
         <visual>
-            <origin xyz="0 0 0" rpy="1.57 0 0" />
+            <origin xyz="-0.02245 0 0" rpy="0 0 0" />
             <geometry>
-                <mesh filename="package://rmitbot_description/meshes/wheel_right_link.STL" />
+                <mesh filename="package://rmitbot_description/meshes/front_left_wheel.stl" scale="0.001 0.001 0.001" />
             </geometry>
         </visual>
         <collision>
-            <origin xyz="0 -0.015 0" rpy="1.57 0 0" />
+            <origin xyz="0 0 0" rpy="0 ${pi/2} 0" />
             <geometry>
-                <sphere radius="0.033"/>
+                <cylinder radius="0.05" length="0.0449"/>
             </geometry>
         </collision>
     </link>
-    <joint name="wheel_right_joint" type="continuous">
-        <origin xyz="0 -0.0701101849418637 0" rpy="0 0 0" />
+    <joint name="front_left_wheel_joint" type="continuous">
+        <origin xyz="-0.18045 0.17 -0.003" rpy="0 0 0" />
         <parent link="base_link" />
-        <child link="wheel_right_link" />
-        <axis xyz="0 1 0" />
+        <child link="front_left_wheel" />
+        <axis xyz="1 0 0" />
     </joint>
-    <link name="wheel_left_link">
+    <link name="rear_left_wheel">
         <inertial>
-            <origin xyz="0 0.014 0" rpy="0 0 0" />
-            <mass value="0.0530086043217644" />
-            <inertia ixx="1.8792911368909E-05" ixy="3.31256392204584E-10" ixz="-1.14082001662767E-08" iyy="3.11510738759073E-05" iyz="-3.60499245082192E-10" izz="1.88266886146847E-05" />
+            <origin xyz="0 0 0" rpy="0 0 0" />
+            <mass value="4.315763" />
+            <inertia
+                ixx="0.0053947033" ixy="-2.274e-12" ixz="0.0"
+                iyy="0.0044596211" iyz="0.0"
+                izz="0.0044596218" />
         </inertial>
         <visual>
-            <origin xyz="0 0 0" rpy="-1.57 0 0" />
+            <origin xyz="-0.02245 0 0" rpy="0 0 0" />
             <geometry>
-                <mesh filename="package://rmitbot_description/meshes/wheel_left_link.STL" />
+                <mesh filename="package://rmitbot_description/meshes/rear_left_wheel.stl" scale="0.001 0.001 0.001"/>
             </geometry>
         </visual>
         <collision>
-            <origin xyz="0 0.015 0" rpy="-1.57 0 0" />
+            <origin xyz="0 0 0" rpy="0 ${pi/2} 0" />
             <geometry>
-                <sphere radius="0.033"/>
+                <cylinder radius="0.05" length="0.0449"/>
             </geometry>
         </collision>
     </link>
-    <joint name="wheel_left_joint" type="continuous">
-        <origin xyz="0 0.0701101849418642 0" rpy="0 0 0" />
+    <joint name="rear_left_wheel_joint" type="continuous">
+        <origin xyz="-0.18045 -0.17 -0.003" rpy="0 0 0" />
         <parent link="base_link" />
-        <child link="wheel_left_link" />
-        <axis xyz="0 1 0" />
+        <child link="rear_left_wheel" />
+        <axis xyz="1 0 0" />
     </joint>
-    <link name="caster_front_link">
+    <link name="front_right_wheel">
         <inertial>
-            <origin xyz="3.89968128948481E-07 2.40073004698083E-07 0.00219173397061506" rpy="0 0 0" />
-            <mass value="1.44379265037903E-06" />
-            <inertia ixx="7.23075276010246E-11" ixy="-6.10956883467859E-16" ixz="2.22849693525031E-15" iyy="3.8713793085917E-11" iyz="2.93909858781952E-15" izz="1.00967486676306E-10" />
+            <origin xyz="0 0 0" rpy="0 0 0" />
+            <mass value="4.315763" />
+            <inertia
+                ixx="0.0053947033" ixy="2.274e-12" ixz="0.0"
+                iyy="0.0044596211" iyz="0.0"
+                izz="0.0044596218" />
         </inertial>
         <visual>
-            <origin xyz="0 0 0" rpy="0 0 0" />
+            <origin xyz="-0.02245 0 0" rpy="0 0 0" />
             <geometry>
-                <mesh filename="package://rmitbot_description/meshes/caster_front_link.STL" />
+                <mesh filename="package://rmitbot_description/meshes/front_right_wheel.stl" scale="0.001 0.001 0.001"/>
             </geometry>
         </visual>
         <collision>
-            <origin xyz="0 0 0" rpy="0 0 0" />
+            <origin xyz="0 0 0" rpy="0 ${pi/2} 0" />
             <geometry>
-                <sphere radius="0.005"/>
+                <cylinder radius="0.05" length="0.0449"/>
             </geometry>
         </collision>
     </link>
-    <joint name="caster_front_joint" type="fixed">
-        <origin xyz="0.04755 0 -0.0275" rpy="0 0 0" />
+    <joint name="front_right_wheel_joint" type="continuous">
+        <origin xyz="0.18045 0.17 -0.003" rpy="0 0 0" />
         <parent link="base_link" />
-        <child link="caster_front_link" />
-        <axis xyz="0 0 0" />
+        <child link="front_right_wheel" />
+        <axis xyz="1 0 0" />
     </joint>
-    <link name="caster_rear_link">
+    <link name="rear_right_wheel">
         <inertial>
-            <origin xyz="3.8996812895542E-07 2.40073004698083E-07 0.00219173397061509" rpy="0 0 0" />
-            <mass value="1.44379265037902E-06" />
-            <inertia ixx="7.23075276010246E-11" ixy="-6.10956872363424E-16" ixz="2.22849693527207E-15" iyy="3.87137930859167E-11" iyz="2.939098587861E-15" izz="1.00967486676306E-10" />
+            <origin xyz="0 0 0" rpy="0 0 0" />
+            <mass value="4.315763" />
+            <inertia
+                ixx="0.0053947033" ixy="-2.274e-12" ixz="0.0"
+                iyy="0.0044596211" iyz="0.0"
+                izz="0.0044596218" />
         </inertial>
         <visual>
-            <origin xyz="0 0 0" rpy="0 0 0" />
+            <origin xyz="-0.02245 0 0" rpy="0 0 0" />
             <geometry>
-                <mesh filename="package://rmitbot_description/meshes/caster_rear_link.STL" />
+                <mesh filename="package://rmitbot_description/meshes/rear_right_wheel.stl" scale="0.001 0.001 0.001"/>
             </geometry>
         </visual>
         <collision>
-            <origin xyz="0 0 0" rpy="0 0 0" />
+            <origin xyz="0 0 0" rpy="0 ${pi/2} 0" />
             <geometry>
-                <sphere radius="0.005"/>
+                <cylinder radius="0.05" length="0.0449"/>
             </geometry>
         </collision>
     </link>
-    <joint name="caster_rear_joint" type="fixed">
-        <origin xyz="-0.04755 0 -0.0275" rpy="0 0 0" />
+    <joint name="rear_right_wheel_joint" type="continuous">
+        <origin xyz="0.18045 -0.17 -0.003" rpy="0 0 0" />
         <parent link="base_link" />
-        <child link="caster_rear_link" />
-        <axis xyz="0 0 0" />
+        <child link="rear_right_wheel" />
+        <axis xyz="1 0 0" />
     </joint>
 </robot>

File: install/rmitbot_description/share/rmitbot_description/urdf/rmitbot_ros2_control.xacro (robot description, xacro)
@@ -1,20 +1,12 @@
 <?xml version="1.0"?>
-<robot xmlns:xacro="http://www.ros.org/wiki/xacro" name="rmitbot">
+<robot name="rmitbot" xmlns:xacro="http://www.ros.org/wiki/xacro" >
+    <!-- ros2_control parameters -->
     <ros2_control name="RobotSystem" type="system">
         <!-- ros2_control Gazebo -->
-        <xacro:if value="$(arg is_sim)">
-            <hardware>
-                <plugin>gz_ros2_control/GazeboSimSystem</plugin>
-            </hardware>
-        </xacro:if>
-        <!-- ros2_control Real Robot -->
-        <xacro:unless value="$(arg is_sim)">
-            <hardware>
-                <plugin>rmitbot_firmware/RmitbotInterface</plugin>
-                <param name="port">/dev/ttyUSB0</param>
-            </hardware>
-        </xacro:unless>
+        <hardware>
+            <plugin>gz_ros2_control/GazeboSimSystem</plugin>
+        </hardware>
         <!-- ros2_control Common Interfaces -->
-        <joint name="wheel_right_joint">
+        <joint name="front_left_wheel_joint">
             <command_interface name="velocity">
                 <param name="min">-1</param>
@@ -24,5 +16,21 @@
             <state_interface name="velocity" />
         </joint>
-        <joint name="wheel_left_joint">
+        <joint name="front_right_wheel_joint">
+            <command_interface name="velocity">
+                <param name="min">-1</param>
+                <param name="max">1</param>
+            </command_interface>
+            <state_interface name="position" />
+            <state_interface name="velocity" />
+        </joint>
+        <joint name="rear_left_wheel_joint">
+            <command_interface name="velocity">
+                <param name="min">-1</param>
+                <param name="max">1</param>
+            </command_interface>
+            <state_interface name="position" />
+            <state_interface name="velocity" />
+        </joint>
+        <joint name="rear_right_wheel_joint">
             <command_interface name="velocity">
                 <param name="min">-1</param>
