Commit message: update code,urdf

File: install/rmitbot_description/share/rmitbot_description/urdf/rmitbot_platform.xacro (robot description, xacro)
@@ -20,4 +20,7 @@
                 <mesh filename="package://rmitbot_description/meshes/base_link.stl" scale="0.001 0.001 0.001"/>
             </geometry>
+            <material name="blue">
+                <color rgba="0 0 1 1"/>
+            </material>
         </visual>
         <collision>
@@ -37,5 +40,32 @@
         <parent link="base_footprint"/>
         <child link="base_link" />
-        <origin xyz="0 0 0.052" rpy="0 0 0"/>
+        <origin xyz="0 0 0.052" rpy="0 0 -${pi/2}"/>
+    </joint>
+    <link name="laser">
+        <inertial>
+            <origin xyz="0 0 0" rpy="0 0 0" />
+            <mass value="0.1" />
+            <inertia ixx="0.0001" ixy="0" ixz="0" iyy="0.0001" iyz="0" izz="0.0001" />
+        </inertial>
+        <visual>
+            <origin xyz="0 0 0" rpy="0 0 0" />
+            <geometry>
+                <cylinder radius="0.05" length="0.1" />
+            </geometry>
+            <material name="green">
+                <color rgba="0 1 0 1" />
+            </material>
+        </visual>
+        <collision>
+            <origin xyz="0 0 0" rpy="0 0 0" />
+            <geometry>
+                <cylinder radius="0.05" length="0.1" />
+            </geometry>
+        </collision>
+    </link>
+    <joint name="laser_joint" type="fixed">
+        <parent link="base_link" />
+        <child link="laser" />
+        <origin xyz="0.15 0.15 0.1" rpy="0.0 0.0 ${pi/2}" />
     </joint>
     <link name="front_left_wheel">
@@ -53,4 +83,7 @@
                 <mesh filename="package://rmitbot_description/meshes/front_left_wheel.stl" scale="0.001 0.001 0.001" />
             </geometry>
+            <material name="black">
+                <color rgba="0 0 0 1"/>
+            </material>
         </visual>
         <collision>
@@ -67,5 +100,5 @@
         <axis xyz="1 0 0" />
     </joint>
-    <link name="rear_left_wheel">
+    <link name="rear_right_wheel">
         <inertial>
             <origin xyz="0 0 0" rpy="0 0 0" />
@@ -81,4 +114,7 @@
                 <mesh filename="package://rmitbot_description/meshes/rear_left_wheel.stl" scale="0.001 0.001 0.001"/>
             </geometry>
+            <material name="black">
+                <color rgba="0 0 0 1"/>
+            </material>
         </visual>
         <collision>
@@ -89,5 +125,5 @@
         </collision>
     </link>
-    <joint name="rear_left_wheel_joint" type="continuous">
+    <joint name="rear_right_wheel_joint" type="continuous">
         <origin xyz="-0.18045 -0.17 -0.003" rpy="0 0 0" />
         <parent link="base_link" />
@@ -109,4 +145,7 @@
                 <mesh filename="package://rmitbot_description/meshes/front_right_wheel.stl" scale="0.001 0.001 0.001"/>
             </geometry>
+            <material name="black">
+                <color rgba="0 0 0 1"/>
+            </material>
         </visual>
         <collision>
@@ -123,5 +162,5 @@
         <axis xyz="1 0 0" />
     </joint>
-    <link name="rear_right_wheel">
+    <link name="rear_left_wheel">
         <inertial>
             <origin xyz="0 0 0" rpy="0 0 0" />
@@ -137,4 +176,7 @@
                 <mesh filename="package://rmitbot_description/meshes/rear_right_wheel.stl" scale="0.001 0.001 0.001"/>
             </geometry>
+            <material name="black">
+                <color rgba="0 0 0 1"/>
+            </material>
         </visual>
         <collision>
@@ -145,5 +187,5 @@
         </collision>
     </link>
-    <joint name="rear_right_wheel_joint" type="continuous">
+    <joint name="rear_left_wheel_joint" type="continuous">
         <origin xyz="0.18045 -0.17 -0.003" rpy="0 0 0" />
         <parent link="base_link" />
